File: hf-transverter-2021/hf-transverter-2021.sch (KiCad schematic (older format))
At the start: 0 parts

Commit message: Adding preselection BPF
Added ELISE designed BPF for the RF input. Placed notes for LO and RF Output filter.
Other:
- note added: "ADD SMA CONNECTOR"
Changed lines of the file:
@@
 Wire Wire Line
 	7200 3675 8325 3675
+Text Notes 1250 3775 0    50   Italic 0
+ADD SMA CONNECTOR
+Text Notes 9800 3700 0    50   Italic 0
+ADD SMA CONNECTOR
 $EndSCHEMATC
