File: hf-transverter-2021/input_rf_filter.sch (KiCad schematic (older format))
At the start: 0 parts

Commit message: Adding preselection BPF
Added ELISE designed BPF for the RF input. Placed notes for LO and RF Output filter.
Parts:
- added C? (x2): 560pF, symbol Device:C
- added C?: 330nH, symbol Device:C
- added L? (x2): 330nH, symbol Device:L
- added L?: 1.5uH, symbol Device:L
Connections:
- new net: C?.2, L?.2
- new net GND: C?.2, C?.2, L?.2, L?.2
- new net RF_INPUT: C?.1, L?.1, L?.1
- new net RF_OUTPUT: C?.1, C?.1, L?.1
Other:
- note added: "3RD ORDER CHEBYSHEV BAND PASS FILTER\nPASSBAND: 9MHz-15MHz"
- note added: "50 OHMS"
Changed lines of the file:
@@
 $Descr A4 11693 8268
 encoding utf-8
-Sheet 1 6
+Sheet 3 6
 Title ""
 Date ""
@@
 Comment4 ""
 $EndDescr
+$Comp
+L Device:C C?
+U 1 1 607834E4
+P 4925 3450
+F 0 "C?" H 5040 3496 50  0000 L CNN
+F 1 "560pF" H 5040 3405 50  0000 L CNN
+F 2 "" H 4963 3300 50  0001 C CNN
+F 3 "~" H 4925 3450 50  0001 C CNN
+	1    4925 3450
+	1    0    0    -1
+$EndComp
+$Comp
+L Device:L L?
+U 1 1 60786CD9
+P 5650 3000
+F 0 "L?" V 5840 3000 50  0000 C CNN
+F 1 "1.5uH" V 5749 3000 50  0000 C CNN
+F 2 "" H 5650 3000 50  0001 C CNN
+F 3 "~" H 5650 3000 50  0001 C CNN
+	1    5650 3000
+	0    -1   -1   0
+$EndComp
+$Comp
+L Device:C C?
+U 1 1 60787409
+P 6150 3000
+F 0 "C?" V 5898 3000 50  0000 C CNN
+F 1 "330nH" V 5989 3000 50  0000 C CNN
+F 2 "" H 6188 2850 50  0001 C CNN
+F 3 "~" H 6150 3000 50  0001 C CNN
+	1    6150 3000
+	0    1    1    0
+$EndComp
+$Comp
+L Device:L L?
+U 1 1 60783D22
+P 4500 3450
+F 0 "L?" H 4552 3496 50  0000 L CNN
+F 1 "330nH" H 4552 3405 50  0000 L CNN
+F 2 "" H 4500 3450 50  0001 C CNN
+F 3 "~" H 4500 3450 50  0001 C CNN
+	1    4500 3450
+	1    0    0    -1
+$EndComp
+Text HLabel 3900 3000 0    50   Input ~ 0
+RF_INPUT
+Text HLabel 7425 3000 2    50   Input ~ 0
+RF_OUTPUT
+$Comp
+L power:GND #PWR?
+U 1 1 607882F9
+P 4500 3750
+F 0 "#PWR?" H 4500 3500 50  0001 C CNN
+F 1 "GND" H 4505 3577 50  0000 C CNN
+F 2 "" H 4500 3750 50  0001 C CNN
+F 3 "" H 4500 3750 50  0001 C CNN
+	1    4500 3750
+	1    0    0    -1
+$EndComp
+$Comp
+L power:GND #PWR?
+U 1 1 607888AF
+P 4925 3750
+F 0 "#PWR?" H 4925 3500 50  0001 C CNN
+F 1 "GND" H 4930 3577 50  0000 C CNN
+F 2 "" H 4925 3750 50  0001 C CNN
+F 3 "" H 4925 3750 50  0001 C CNN
+	1    4925 3750
+	1    0    0    -1
+$EndComp
+Wire Wire Line
+	4500 3600 4500 3750
+Wire Wire Line
+	4925 3600 4925 3750
+Wire Wire Line
+	4925 3300 4925 3000
+Wire Wire Line
+	4925 3000 4500 3000
+Wire Wire Line
+	4500 3000 4500 3300
+Wire Wire Line
+	4500 3000 3900 3000
+Connection ~ 4500 3000
+Wire Wire Line
+	4925 3000 5500 3000
+Connection ~ 4925 3000
+Wire Wire Line
+	5800 3000 6000 3000
+$Comp
+L Device:C C?
+U 1 1 6078D13C
+P 7150 3450
+F 0 "C?" H 7265 3496 50  0000 L CNN
+F 1 "560pF" H 7265 3405 50  0000 L CNN
+F 2 "" H 7188 3300 50  0001 C CNN
+F 3 "~" H 7150 3450 50  0001 C CNN
+	1    7150 3450
+	1    0    0    -1
+$EndComp
+$Comp
+L Device:L L?
+U 1 1 6078D142
+P 6725 3450
+F 0 "L?" H 6777 3496 50  0000 L CNN
+F 1 "330nH" H 6777 3405 50  0000 L CNN
+F 2 "" H 6725 3450 50  0001 C CNN
+F 3 "~" H 6725 3450 50  0001 C CNN
+	1    6725 3450
+	1    0    0    -1
+$EndComp
+$Comp
+L power:GND #PWR?
+U 1 1 6078D148
+P 6725 3750
+F 0 "#PWR?" H 6725 3500 50  0001 C CNN
+F 1 "GND" H 6730 3577 50  0000 C CNN
+F 2 "" H 6725 3750 50  0001 C CNN
+F 3 "" H 6725 3750 50  0001 C CNN
+	1    6725 3750
+	1    0    0    -1
+$EndComp
+$Comp
+L power:GND #PWR?
+U 1 1 6078D14E
+P 7150 3750
+F 0 "#PWR?" H 7150 3500 50  0001 C CNN
+F 1 "GND" H 7155 3577 50  0000 C CNN
+F 2 "" H 7150 3750 50  0001 C CNN
+F 3 "" H 7150 3750 50  0001 C CNN
+	1    7150 3750
+	1    0    0    -1
+$EndComp
+Wire Wire Line
+	6725 3600 6725 3750
+Wire Wire Line
+	7150 3600 7150 3750
+Wire Wire Line
+	7150 3300 7150 3000
+Wire Wire Line
+	7150 3000 6725 3000
+Wire Wire Line
+	6725 3000 6725 3300
+Connection ~ 6725 3000
+Wire Wire Line
+	7150 3000 7425 3000
+Connection ~ 7150 3000
+Wire Wire Line
+	6300 3000 6725 3000
+Text Notes 5100 4475 0    50   ~ 0
+3RD ORDER CHEBYSHEV BAND PASS FILTER\nPASSBAND: 9MHz-15MHz
+Text Notes 3975 2925 0    50   ~ 0
+50 OHMS
+Text Notes 7000 2925 0    50   ~ 0
+50 OHMS
 $EndSCHEMATC
