File: hf-transverter-2021/local_oscillator.sch (KiCad schematic (older format))
At the start: 0 parts

Commit message: Adding preselection BPF
Added ELISE designed BPF for the RF input. Placed notes for LO and RF Output filter.
Other:
- note added: "PLACE LPF TO AVOID HARMONICS"
Changed lines of the file:
@@
 $Descr A4 11693 8268
 encoding utf-8
-Sheet 1 6
+Sheet 4 6
 Title ""
 Date ""
@@
 Comment4 ""
 $EndDescr
+Text Notes 6825 3000 0    50   Italic 0
+PLACE LPF TO AVOID HARMONICS
 $EndSCHEMATC
