File: hf-transverter-2021/output_rf_filter.sch (KiCad schematic (older format))
At the start: 0 parts

Commit message: Adding preselection BPF
Added ELISE designed BPF for the RF input. Placed notes for LO and RF Output filter.
Other:
- note added: "PLACE EITHER HPF OR BANDPASS FILTER"
Changed lines of the file:
@@
 $Descr A4 11693 8268
 encoding utf-8
-Sheet 1 6
+Sheet 6 6
 Title ""
 Date ""
@@
 Comment4 ""
 $EndDescr
+Text Notes 6475 1450 0    50   Italic 0
+PLACE EITHER HPF OR BANDPASS FILTER
 $EndSCHEMATC
